Commit message: lidar working

File: rover_description/urdf/bases/turnbuckle.urdf.xacro (robot description, xacro)
@@ -62,4 +62,5 @@
                 </inertial>
             </link>
+            <!-- can't have closed loops in URDF
             <joint name="back_${lat_label}_turnbuckle_joint" type="ball">
                 <pose>-0.035 0 0 0 0 0</pose>
@@ -67,4 +68,5 @@
                 <child>${lat_label}_turnbuckle_link</child>
             </joint>
+            -->
             <joint name="front_${lat_label}_turnbuckle_joint" type="ball">
                 <pose>0.035 0 0 0 0 0</pose>

File: rover_description/urdf/sensors/asus_xtion.urdf.xacro (robot description, xacro)
@@ -61,4 +61,5 @@
       </inertial>
     </link>
+<!--
     <gazebo reference="${prefix}_link">
       <sensor name="camera" type="depth">
@@ -150,4 +151,5 @@
       </sensor>
     </gazebo>
+-->
   </xacro:macro>
 </robot>

File: rover_description/urdf/sensors/hokuyo.urdf.xacro (robot description, xacro)
@@ -46,6 +46,4 @@
       <material>Gazebo/DarkGrey</material>
     </gazebo>
-    <link name="${prefix}_link">
-    </link>
     <joint name="${prefix}_joint" type="fixed">
       <parent link="${prefix}_base_link"/>
@@ -53,11 +51,20 @@
       <origin xyz="0.00 0 0.0" rpy="0 0 0"/>
     </joint>
-<!--
+    <link name="${prefix}_link">
+    </link>
+    <gazebo>
+      <plugin
+          filename="gz-sim-sensors-system"
+          name="gz::sim::systems::Sensors">
+          <render_engine>ogre2</render_engine>
+      </plugin>
+    </gazebo>
     <gazebo reference="${prefix}_link">
-    <sensor name='gpu_lidar' type='gpu_lidar'>"
-    <pose relative_to="${prefix}_link">0 0 0 0 0 0</pose>
-    <topic>scan</topic>
-    <update_rate>10</update_rate>
-    <ray>
+      <sensor name='gpu_lidar' type='gpu_lidar'>
+      <pose relative_to='${prefix}_link'>0 0 0 0 0 0</pose>
+      <topic>scan</topic>
+      <gz_frame_id>${prefix}_link</gz_frame_id>
+      <update_rate>10</update_rate>
+      <lidar>
         <scan>
             <horizontal>
@@ -79,10 +86,14 @@
             <resolution>0.01</resolution>
         </range>
-    </ray>
-    <always_on>1</always_on>
+    </lidar>
     <visualize>true</visualize>
-</sensor>
-    </gazebo>
--->
+    </sensor>
+  </gazebo>
+  <gazebo>
+    <plugin name="gz::sim::systems::LidarVisual"
+        filename="gz-sim-lidar-visual-system">
+        <topic>/scan</topic>
+    </plugin>
+  </gazebo>
   </xacro:macro>
 </robot>
