Commit message: useless

File: rover_description/models/rover.urdf.xacro (robot description, xacro)
@@ -12,190 +12,4 @@
     <xacro:include filename="$(find rover_description)/urdf/wheels/corner.urdf.xacro" />
     <xacro:include filename="$(find rover_description)/urdf/sensors/all_sensors.urdf.xacro" />
-    <!-- Gazebo ROS2 Control
-    <gazebo>
-        <plugin filename="libgazebo_ros2_control.so" name="gazebo_ros2_control">
-            <parameters>$(find rover_description)/config/control.yaml</parameters>
-        </plugin>
-    </gazebo>
-    <gazebo>
-        <plugin name="rover_joint_state" filename="libgazebo_ros_joint_state_publisher.so">
-            <update_rate>30</update_rate>
-            <joint_name>left_rocker_joint</joint_name>
-            <joint_name>right_rocker_joint</joint_name>
-            <joint_name>left_bogie_joint</joint_name>
-            <joint_name>right_bogie_joint</joint_name>
-            <joint_name>diff_brace_joint</joint_name>
-            <joint_name>back_left_turnbuckle_joint</joint_name>
-            <joint_name>back_right_turnbuckle_joint</joint_name>
-            <joint_name>front_left_turnbuckle_joint</joint_name>
-            <joint_name>front_right_turnbuckle_joint</joint_name>
-            <joint_name>front_left_corner_joint</joint_name>
-            <joint_name>front_right_corner_joint</joint_name>
-            <joint_name>back_left_corner_joint</joint_name>
-            <joint_name>back_right_corner_joint</joint_name>
-        </plugin>
-    </gazebo>
-    <ros2_control name="GazeboSystem" type="system">
-        <hardware>
-            <plugin>gazebo_ros2_control/GazeboSystem</plugin>
-        </hardware>
-        <joint name="front_right_corner_joint">
-            <command_interface name="position">
-                <param name="min">-3.14159</param>
-                <param name="max">3.14159</param>
-            </command_interface>
-            <state_interface name="position">
-                <param name="initial_value">0.0</param>
-            </state_interface>
-            <state_interface name="velocity"/>
-            <state_interface name="effort"/>
-        </joint>
-        <joint name="front_left_corner_joint">
-            <command_interface name="position">
-                <param name="min">-3.14159</param>
-                <param name="max">3.14159</param>
-            </command_interface>
-            <state_interface name="position">
-                <param name="initial_value">0.0</param>
-            </state_interface>
-            <state_interface name="velocity"/>
-            <state_interface name="effort"/>
-        </joint>
-        <joint name="back_right_corner_joint">
-            <command_interface name="position">
-                <param name="min">-3.14159</param>
-                <param name="max">3.14159</param>
-            </command_interface>
-            <state_interface name="position">
-                <param name="initial_value">0.0</param>
-            </state_interface>
-            <state_interface name="velocity"/>
-            <state_interface name="effort"/>
-        </joint>
-        <joint name="back_left_corner_joint">
-            <command_interface name="position">
-                <param name="min">-3.14159</param>
-                <param name="max">3.14159</param>
-            </command_interface>
-            <state_interface name="position">
-                <param name="initial_value">0.0</param>
-            </state_interface>
-            <state_interface name="velocity"/>
-            <state_interface name="effort"/>
-        </joint>
-        <joint name="front_right_wheel_joint">
-            <command_interface name="velocity">
-                <param name="min">-10</param>
-                <param name="max">10</param>
-            </command_interface>
-            <state_interface name="position"/>
-            <state_interface name="velocity"/>
-            <state_interface name="effort"/>
-        </joint>
-        <joint name="front_left_wheel_joint">
-            <command_interface name="velocity">
-                <param name="min">-10</param>
-                <param name="max">10</param>
-            </command_interface>
-            <state_interface name="position"/>
-            <state_interface name="velocity"/>
-            <state_interface name="effort"/>
-        </joint>
-        <joint name="mid_right_wheel_joint">
-            <command_interface name="velocity">
-                <param name="min">-10</param>
-                <param name="max">10</param>
-            </command_interface>
-            <state_interface name="position"/>
-            <state_interface name="velocity"/>
-            <state_interface name="effort"/>
-        </joint>
-        <joint name="mid_left_wheel_joint">
-            <command_interface name="velocity">
-                <param name="min">-10</param>
-                <param name="max">10</param>
-            </command_interface>
-            <state_interface name="position"/>
-            <state_interface name="velocity"/>
-            <state_interface name="effort"/>
-        </joint>
-        <joint name="back_right_wheel_joint">
-            <command_interface name="velocity">
-                <param name="min">-10</param>
-                <param name="max">10</param>
-            </command_interface>
-            <state_interface name="position"/>
-            <state_interface name="velocity"/>
-            <state_interface name="effort"/>
-        </joint>
-        <joint name="back_left_wheel_joint">
-            <command_interface name="velocity">
-                <param name="min">-10</param>
-                <param name="max">10</param>
-            </command_interface>
-            <state_interface name="position"/>
-            <state_interface name="velocity"/>
-            <state_interface name="effort"/>
-        </joint>
-    </ros2_control>
-    -->
-<!-- Plugin config from https://github.com/ThiwakarS/ROS2-jazzy-GZ-harmonic -->
-<!--
-<gazebo>
-        <plugin
-            filename="gz-sim-user-commands-system"
-            name="gz::sim::systems::UserCommands">
-        </plugin>
-        <plugin
-            filename="gz-sim-scene-broadcaster-system"
-            name="gz::sim::systems::SceneBroadcaster">
-        </plugin>
-        <plugin
-            filename="gz-sim-sensors-system"
-            name="gz::sim::systems::Sensors">
-            <render_engine>ogre2</render_engine>
-        </plugin>
-        <plugin
-            filename="gz-sim-imu-system"
-            name="gz::sim::systems::Imu">
-        </plugin>
-    </gazebo>
--->
-    <!-- Temporary
-        <plugin
-            filename="gz-sim-diff-drive-system"
-            name="gz::sim::systems::DiffDrive">
-            <left_joint>mid_left_wheel_joint</left_joint>
-            <right_joint>mid_right_wheel_joint</right_joint>
-            <wheel_separation>0.0929</wheel_separation>
-            <wheel_radius>0.06</wheel_radius>
-            <topic>cmd_vel</topic>
-            <odom_topic>odom</odom_topic>
-            <frame_id>odom</frame_id>
-            <child_frame_id>base_link</child_frame_id>
-            <odom_publisher_frequency>50</odom_publisher_frequency>
-            <tf_topic>/tf</tf_topic>
-        </plugin>
-        <plugin filename="gz-sim-joint-state-publisher-system"
-            name="gz::sim::systems::JointStatePublisher">
-            <topic>joint_states</topic>
-            <joint_name>left_rocker_joint</joint_name>
-            <joint_name>right_rocker_joint</joint_name>
-            <joint_name>left_bogie_joint</joint_name>
-            <joint_name>right_bogie_joint</joint_name>
-            <joint_name>diff_brace_joint</joint_name>
-            <joint_name>back_left_turnbuckle_joint</joint_name>
-            <joint_name>back_right_turnbuckle_joint</joint_name>
-            <joint_name>front_left_turnbuckle_joint</joint_name>
-            <joint_name>front_right_turnbuckle_joint</joint_name>
-            <joint_name>front_left_corner_joint</joint_name>
-            <joint_name>front_right_corner_joint</joint_name>
-            <joint_name>back_left_corner_joint</joint_name>
-            <joint_name>back_right_corner_joint</joint_name>
-        </plugin>
-        <plugin filename="libgazebo_ros2_control.so" name="gazebo_ros2_control">
-            <parameters>$(find rover_description)/config/control.yaml</parameters>
-        </plugin>
--->
     <!-- The base link -->
     <link name="base_link">
@@ -253,3 +67,189 @@
     <xacro:corner_wheel_joint lon_label="back" lat_label="left" reflect="1"/>
     <xacro:corner_wheel_joint lon_label="back" lat_label="right" reflect="-1"/>
+    <!-- Gazebo ROS2 Control
+    <gazebo>
+        <plugin filename="libgazebo_ros2_control.so" name="gazebo_ros2_control">
+            <parameters>$(find rover_description)/config/control.yaml</parameters>
+        </plugin>
+    </gazebo>
+    <gazebo>
+        <plugin name="rover_joint_state" filename="libgazebo_ros_joint_state_publisher.so">
+            <update_rate>30</update_rate>
+            <joint_name>left_rocker_joint</joint_name>
+            <joint_name>right_rocker_joint</joint_name>
+            <joint_name>left_bogie_joint</joint_name>
+            <joint_name>right_bogie_joint</joint_name>
+            <joint_name>diff_brace_joint</joint_name>
+            <joint_name>back_left_turnbuckle_joint</joint_name>
+            <joint_name>back_right_turnbuckle_joint</joint_name>
+            <joint_name>front_left_turnbuckle_joint</joint_name>
+            <joint_name>front_right_turnbuckle_joint</joint_name>
+            <joint_name>front_left_corner_joint</joint_name>
+            <joint_name>front_right_corner_joint</joint_name>
+            <joint_name>back_left_corner_joint</joint_name>
+            <joint_name>back_right_corner_joint</joint_name>
+        </plugin>
+    </gazebo>
+    <ros2_control name="GazeboSystem" type="system">
+        <hardware>
+            <plugin>gazebo_ros2_control/GazeboSystem</plugin>
+        </hardware>
+        <joint name="front_right_corner_joint">
+            <command_interface name="position">
+                <param name="min">-3.14159</param>
+                <param name="max">3.14159</param>
+            </command_interface>
+            <state_interface name="position">
+                <param name="initial_value">0.0</param>
+            </state_interface>
+            <state_interface name="velocity"/>
+            <state_interface name="effort"/>
+        </joint>
+        <joint name="front_left_corner_joint">
+            <command_interface name="position">
+                <param name="min">-3.14159</param>
+                <param name="max">3.14159</param>
+            </command_interface>
+            <state_interface name="position">
+                <param name="initial_value">0.0</param>
+            </state_interface>
+            <state_interface name="velocity"/>
+            <state_interface name="effort"/>
+        </joint>
+        <joint name="back_right_corner_joint">
+            <command_interface name="position">
+                <param name="min">-3.14159</param>
+                <param name="max">3.14159</param>
+            </command_interface>
+            <state_interface name="position">
+                <param name="initial_value">0.0</param>
+            </state_interface>
+            <state_interface name="velocity"/>
+            <state_interface name="effort"/>
+        </joint>
+        <joint name="back_left_corner_joint">
+            <command_interface name="position">
+                <param name="min">-3.14159</param>
+                <param name="max">3.14159</param>
+            </command_interface>
+            <state_interface name="position">
+                <param name="initial_value">0.0</param>
+            </state_interface>
+            <state_interface name="velocity"/>
+            <state_interface name="effort"/>
+        </joint>
+        <joint name="front_right_wheel_joint">
+            <command_interface name="velocity">
+                <param name="min">-10</param>
+                <param name="max">10</param>
+            </command_interface>
+            <state_interface name="position"/>
+            <state_interface name="velocity"/>
+            <state_interface name="effort"/>
+        </joint>
+        <joint name="front_left_wheel_joint">
+            <command_interface name="velocity">
+                <param name="min">-10</param>
+                <param name="max">10</param>
+            </command_interface>
+            <state_interface name="position"/>
+            <state_interface name="velocity"/>
+            <state_interface name="effort"/>
+        </joint>
+        <joint name="mid_right_wheel_joint">
+            <command_interface name="velocity">
+                <param name="min">-10</param>
+                <param name="max">10</param>
+            </command_interface>
+            <state_interface name="position"/>
+            <state_interface name="velocity"/>
+            <state_interface name="effort"/>
+        </joint>
+        <joint name="mid_left_wheel_joint">
+            <command_interface name="velocity">
+                <param name="min">-10</param>
+                <param name="max">10</param>
+            </command_interface>
+            <state_interface name="position"/>
+            <state_interface name="velocity"/>
+            <state_interface name="effort"/>
+        </joint>
+        <joint name="back_right_wheel_joint">
+            <command_interface name="velocity">
+                <param name="min">-10</param>
+                <param name="max">10</param>
+            </command_interface>
+            <state_interface name="position"/>
+            <state_interface name="velocity"/>
+            <state_interface name="effort"/>
+        </joint>
+        <joint name="back_left_wheel_joint">
+            <command_interface name="velocity">
+                <param name="min">-10</param>
+                <param name="max">10</param>
+            </command_interface>
+            <state_interface name="position"/>
+            <state_interface name="velocity"/>
+            <state_interface name="effort"/>
+        </joint>
+    </ros2_control>
+    -->
+<!-- Plugin config from https://github.com/ThiwakarS/ROS2-jazzy-GZ-harmonic -->
+<!--
+<gazebo>
+        <plugin
+            filename="gz-sim-user-commands-system"
+            name="gz::sim::systems::UserCommands">
+        </plugin>
+        <plugin
+            filename="gz-sim-scene-broadcaster-system"
+            name="gz::sim::systems::SceneBroadcaster">
+        </plugin>
+        <plugin
+            filename="gz-sim-sensors-system"
+            name="gz::sim::systems::Sensors">
+            <render_engine>ogre2</render_engine>
+        </plugin>
+        <plugin
+            filename="gz-sim-imu-system"
+            name="gz::sim::systems::Imu">
+        </plugin>
+    </gazebo>
+-->
+    <!-- Temporary
+        <plugin
+            filename="gz-sim-diff-drive-system"
+            name="gz::sim::systems::DiffDrive">
+            <left_joint>mid_left_wheel_joint</left_joint>
+            <right_joint>mid_right_wheel_joint</right_joint>
+            <wheel_separation>0.0929</wheel_separation>
+            <wheel_radius>0.06</wheel_radius>
+            <topic>cmd_vel</topic>
+            <odom_topic>odom</odom_topic>
+            <frame_id>odom</frame_id>
+            <child_frame_id>base_link</child_frame_id>
+            <odom_publisher_frequency>50</odom_publisher_frequency>
+            <tf_topic>/tf</tf_topic>
+        </plugin>
+        <plugin filename="gz-sim-joint-state-publisher-system"
+            name="gz::sim::systems::JointStatePublisher">
+            <topic>joint_states</topic>
+            <joint_name>left_rocker_joint</joint_name>
+            <joint_name>right_rocker_joint</joint_name>
+            <joint_name>left_bogie_joint</joint_name>
+            <joint_name>right_bogie_joint</joint_name>
+            <joint_name>diff_brace_joint</joint_name>
+            <joint_name>back_left_turnbuckle_joint</joint_name>
+            <joint_name>back_right_turnbuckle_joint</joint_name>
+            <joint_name>front_left_turnbuckle_joint</joint_name>
+            <joint_name>front_right_turnbuckle_joint</joint_name>
+            <joint_name>front_left_corner_joint</joint_name>
+            <joint_name>front_right_corner_joint</joint_name>
+            <joint_name>back_left_corner_joint</joint_name>
+            <joint_name>back_right_corner_joint</joint_name>
+        </plugin>
+        <plugin filename="libgazebo_ros2_control.so" name="gazebo_ros2_control">
+            <parameters>$(find rover_description)/config/control.yaml</parameters>
+        </plugin>
+-->
 </robot>

File: rover_description/urdf/sensors/hokuyo.urdf.xacro (robot description, xacro)
@@ -90,10 +90,4 @@
     </sensor>
   </gazebo>
-  <gazebo>
-    <plugin name="gz::sim::systems::LidarVisual"
-        filename="gz-sim-lidar-visual-system">
-        <topic>/scan</topic>
-    </plugin>
-  </gazebo>
   </xacro:macro>
 </robot>
