Commit message: updating URDF for simulation

File: rover_description/models/rover.urdf.xacro (robot description, xacro)
@@ -12,4 +12,9 @@
     <xacro:include filename="$(find rover_description)/urdf/wheels/corner.urdf.xacro" />
     <xacro:include filename="$(find rover_description)/urdf/sensors/all_sensors.urdf.xacro" />
+    <!-- enables slightly differnt physics for simulation and control -->
+    <!-- TODO: figure out how to set this to false when not in simulation - we don't seem to be running
+               robot_state_publisher on the real robot? -->
+    <!-- do we even need this since we set it to default to true in rocker & turnbuckle? -->
+    <xacro:property name="use_gazebo" value="true"/>
     <!-- The base link -->
     <link name="base_link">
@@ -29,4 +34,5 @@
     <xacro:differential parent="base_link" />
     <xacro:turnbuckle lat_label="left" reflect="1"/>
+    <!--
     <xacro:turnbuckle lat_label="right" reflect="-1"/>
     <xacro:rocker parent="base_link" lat_label="left" reflect="1"/>
@@ -34,17 +40,13 @@
     <xacro:bogie lat_label="left" reflect="1"/>
     <xacro:bogie lat_label="right" reflect="-1"/>
-    <!-- sensors -->
     <xacro:sensor_hokuyo prefix="laser" parent="base_link" min_angle="-1.0" max_angle="1.0">
         <origin xyz="0.17 0 0.005" rpy="0 0 0"/>
     </xacro:sensor_hokuyo>
     <xacro:sensor_imu prefix="imu" parent="base_link">
-        <!-- <origin xyz="-0.32 0 0.05" rpy="0 0.5 0"/> -->
         <origin xyz="0 0 -0.04" rpy="0 0 0"/>
     </xacro:sensor_imu>
     <xacro:sensor_asus_xtion prefix="camera" parent="base_link">
         <origin xyz="0.215 0 0.065" rpy="0 0.4 0"/>
-        <!-- <origin xyz="0.212 0 0.065" rpy="0 0 0"/> -->
     </xacro:sensor_asus_xtion>
-    <!-- wheels -->
     <xacro:corner_link lon_label="front" lat_label="left" reflect="1"/>
     <xacro:corner_link lon_label="front" lat_label="right" reflect="-1"/>
@@ -67,169 +69,8 @@
     <xacro:corner_wheel_joint lon_label="back" lat_label="left" reflect="1"/>
     <xacro:corner_wheel_joint lon_label="back" lat_label="right" reflect="-1"/>
-    <!-- Gazebo ROS2 Control
+    -->
+    <!-- For Gazebo Harmonic (Ignition/Gazebo >= Garden), use gz-sim-joint-state-publisher-system -->
+    <!--
     <gazebo>
-        <plugin filename="libgazebo_ros2_control.so" name="gazebo_ros2_control">
-            <parameters>$(find rover_description)/config/control.yaml</parameters>
-        </plugin>
-    </gazebo>
-    <gazebo>
-        <plugin name="rover_joint_state" filename="libgazebo_ros_joint_state_publisher.so">
-            <update_rate>30</update_rate>
-            <joint_name>left_rocker_joint</joint_name>
-            <joint_name>right_rocker_joint</joint_name>
-            <joint_name>left_bogie_joint</joint_name>
-            <joint_name>right_bogie_joint</joint_name>
-            <joint_name>diff_brace_joint</joint_name>
-            <joint_name>back_left_turnbuckle_joint</joint_name>
-            <joint_name>back_right_turnbuckle_joint</joint_name>
-            <joint_name>front_left_turnbuckle_joint</joint_name>
-            <joint_name>front_right_turnbuckle_joint</joint_name>
-            <joint_name>front_left_corner_joint</joint_name>
-            <joint_name>front_right_corner_joint</joint_name>
-            <joint_name>back_left_corner_joint</joint_name>
-            <joint_name>back_right_corner_joint</joint_name>
-        </plugin>
-    </gazebo>
-    <ros2_control name="GazeboSystem" type="system">
-        <hardware>
-            <plugin>gazebo_ros2_control/GazeboSystem</plugin>
-        </hardware>
-        <joint name="front_right_corner_joint">
-            <command_interface name="position">
-                <param name="min">-3.14159</param>
-                <param name="max">3.14159</param>
-            </command_interface>
-            <state_interface name="position">
-                <param name="initial_value">0.0</param>
-            </state_interface>
-            <state_interface name="velocity"/>
-            <state_interface name="effort"/>
-        </joint>
-        <joint name="front_left_corner_joint">
-            <command_interface name="position">
-                <param name="min">-3.14159</param>
-                <param name="max">3.14159</param>
-            </command_interface>
-            <state_interface name="position">
-                <param name="initial_value">0.0</param>
-            </state_interface>
-            <state_interface name="velocity"/>
-            <state_interface name="effort"/>
-        </joint>
-        <joint name="back_right_corner_joint">
-            <command_interface name="position">
-                <param name="min">-3.14159</param>
-                <param name="max">3.14159</param>
-            </command_interface>
-            <state_interface name="position">
-                <param name="initial_value">0.0</param>
-            </state_interface>
-            <state_interface name="velocity"/>
-            <state_interface name="effort"/>
-        </joint>
-        <joint name="back_left_corner_joint">
-            <command_interface name="position">
-                <param name="min">-3.14159</param>
-                <param name="max">3.14159</param>
-            </command_interface>
-            <state_interface name="position">
-                <param name="initial_value">0.0</param>
-            </state_interface>
-            <state_interface name="velocity"/>
-            <state_interface name="effort"/>
-        </joint>
-        <joint name="front_right_wheel_joint">
-            <command_interface name="velocity">
-                <param name="min">-10</param>
-                <param name="max">10</param>
-            </command_interface>
-            <state_interface name="position"/>
-            <state_interface name="velocity"/>
-            <state_interface name="effort"/>
-        </joint>
-        <joint name="front_left_wheel_joint">
-            <command_interface name="velocity">
-                <param name="min">-10</param>
-                <param name="max">10</param>
-            </command_interface>
-            <state_interface name="position"/>
-            <state_interface name="velocity"/>
-            <state_interface name="effort"/>
-        </joint>
-        <joint name="mid_right_wheel_joint">
-            <command_interface name="velocity">
-                <param name="min">-10</param>
-                <param name="max">10</param>
-            </command_interface>
-            <state_interface name="position"/>
-            <state_interface name="velocity"/>
-            <state_interface name="effort"/>
-        </joint>
-        <joint name="mid_left_wheel_joint">
-            <command_interface name="velocity">
-                <param name="min">-10</param>
-                <param name="max">10</param>
-            </command_interface>
-            <state_interface name="position"/>
-            <state_interface name="velocity"/>
-            <state_interface name="effort"/>
-        </joint>
-        <joint name="back_right_wheel_joint">
-            <command_interface name="velocity">
-                <param name="min">-10</param>
-                <param name="max">10</param>
-            </command_interface>
-            <state_interface name="position"/>
-            <state_interface name="velocity"/>
-            <state_interface name="effort"/>
-        </joint>
-        <joint name="back_left_wheel_joint">
-            <command_interface name="velocity">
-                <param name="min">-10</param>
-                <param name="max">10</param>
-            </command_interface>
-            <state_interface name="position"/>
-            <state_interface name="velocity"/>
-            <state_interface name="effort"/>
-        </joint>
-    </ros2_control>
-    -->
-<!-- Plugin config from https://github.com/ThiwakarS/ROS2-jazzy-GZ-harmonic -->
-<!--
-<gazebo>
-        <plugin
-            filename="gz-sim-user-commands-system"
-            name="gz::sim::systems::UserCommands">
-        </plugin>
-        <plugin
-            filename="gz-sim-scene-broadcaster-system"
-            name="gz::sim::systems::SceneBroadcaster">
-        </plugin>
-        <plugin
-            filename="gz-sim-sensors-system"
-            name="gz::sim::systems::Sensors">
-            <render_engine>ogre2</render_engine>
-        </plugin>
-        <plugin
-            filename="gz-sim-imu-system"
-            name="gz::sim::systems::Imu">
-        </plugin>
-    </gazebo>
--->
-    <!-- Temporary
-        <plugin
-            filename="gz-sim-diff-drive-system"
-            name="gz::sim::systems::DiffDrive">
-            <left_joint>mid_left_wheel_joint</left_joint>
-            <right_joint>mid_right_wheel_joint</right_joint>
-            <wheel_separation>0.0929</wheel_separation>
-            <wheel_radius>0.06</wheel_radius>
-            <topic>cmd_vel</topic>
-            <odom_topic>odom</odom_topic>
-            <frame_id>odom</frame_id>
-            <child_frame_id>base_link</child_frame_id>
-            <odom_publisher_frequency>50</odom_publisher_frequency>
-            <tf_topic>/tf</tf_topic>
-        </plugin>
         <plugin filename="gz-sim-joint-state-publisher-system"
             name="gz::sim::systems::JointStatePublisher">
@@ -249,4 +90,168 @@
             <joint_name>back_right_corner_joint</joint_name>
         </plugin>
+    </gazebo>
+    -->
+  <gazebo>
+    <plugin filename="gz_ros2_control-system" name="gz_ros2_control::GazeboSimROS2ControlPlugin">
+      <parameters>$(find rover_description)/config/control.yaml</parameters>
+    </plugin>
+  </gazebo>
+    <ros2_control name="RoverSystem" type="system">
+        <hardware>
+            <plugin>gz_ros2_control/GazeboSimSystem</plugin>
+        </hardware>
+        <joint name="front_right_corner_joint">
+            <command_interface name="position">
+                <param name="min">-3.14159</param>
+                <param name="max">3.14159</param>
+            </command_interface>
+            <state_interface name="position">
+                <param name="initial_value">0.0</param>
+            </state_interface>
+            <state_interface name="velocity"/>
+            <state_interface name="effort"/>
+        </joint>
+        <joint name="front_left_corner_joint">
+            <command_interface name="position">
+                <param name="min">-3.14159</param>
+                <param name="max">3.14159</param>
+            </command_interface>
+            <state_interface name="position">
+                <param name="initial_value">0.0</param>
+            </state_interface>
+            <state_interface name="velocity"/>
+            <state_interface name="effort"/>
+        </joint>
+        <joint name="back_right_corner_joint">
+            <command_interface name="position">
+                <param name="min">-3.14159</param>
+                <param name="max">3.14159</param>
+            </command_interface>
+            <state_interface name="position">
+                <param name="initial_value">0.0</param>
+            </state_interface>
+            <state_interface name="velocity"/>
+            <state_interface name="effort"/>
+        </joint>
+        <joint name="back_left_corner_joint">
+            <command_interface name="position">
+                <param name="min">-3.14159</param>
+                <param name="max">3.14159</param>
+            </command_interface>
+            <state_interface name="position">
+                <param name="initial_value">0.0</param>
+            </state_interface>
+            <state_interface name="velocity"/>
+            <state_interface name="effort"/>
+        </joint>
+        <joint name="front_right_wheel_joint">
+            <command_interface name="velocity">
+                <param name="min">-10</param>
+                <param name="max">10</param>
+            </command_interface>
+            <state_interface name="position"/>
+            <state_interface name="velocity"/>
+            <state_interface name="effort"/>
+        </joint>
+        <joint name="front_left_wheel_joint">
+            <command_interface name="velocity">
+                <param name="min">-10</param>
+                <param name="max">10</param>
+            </command_interface>
+            <state_interface name="position"/>
+            <state_interface name="velocity"/>
+            <state_interface name="effort"/>
+        </joint>
+        <joint name="mid_right_wheel_joint">
+            <command_interface name="velocity">
+                <param name="min">-10</param>
+                <param name="max">10</param>
+            </command_interface>
+            <state_interface name="position"/>
+            <state_interface name="velocity"/>
+            <state_interface name="effort"/>
+        </joint>
+        <joint name="mid_left_wheel_joint">
+            <command_interface name="velocity">
+                <param name="min">-10</param>
+                <param name="max">10</param>
+            </command_interface>
+            <state_interface name="position"/>
+            <state_interface name="velocity"/>
+            <state_interface name="effort"/>
+        </joint>
+        <joint name="back_right_wheel_joint">
+            <command_interface name="velocity">
+                <param name="min">-10</param>
+                <param name="max">10</param>
+            </command_interface>
+            <state_interface name="position"/>
+            <state_interface name="velocity"/>
+            <state_interface name="effort"/>
+        </joint>
+        <joint name="back_left_wheel_joint">
+            <command_interface name="velocity">
+                <param name="min">-10</param>
+                <param name="max">10</param>
+            </command_interface>
+            <state_interface name="position"/>
+            <state_interface name="velocity"/>
+            <state_interface name="effort"/>
+        </joint>
+    </ros2_control>
+<!-- Plugin config from https://github.com/ThiwakarS/ROS2-jazzy-GZ-harmonic -->
+<!--
+<gazebo>
+        <plugin
+            filename="gz-sim-user-commands-system"
+            name="gz::sim::systems::UserCommands">
+        </plugin>
+        <plugin
+            filename="gz-sim-scene-broadcaster-system"
+            name="gz::sim::systems::SceneBroadcaster">
+        </plugin>
+        <plugin
+            filename="gz-sim-sensors-system"
+            name="gz::sim::systems::Sensors">
+            <render_engine>ogre2</render_engine>
+        </plugin>
+        <plugin
+            filename="gz-sim-imu-system"
+            name="gz::sim::systems::Imu">
+        </plugin>
+    </gazebo>
+-->
+    <!-- Temporary
+        <plugin
+            filename="gz-sim-diff-drive-system"
+            name="gz::sim::systems::DiffDrive">
+            <left_joint>mid_left_wheel_joint</left_joint>
+            <right_joint>mid_right_wheel_joint</right_joint>
+            <wheel_separation>0.0929</wheel_separation>
+            <wheel_radius>0.06</wheel_radius>
+            <topic>cmd_vel</topic>
+            <odom_topic>odom</odom_topic>
+            <frame_id>odom</frame_id>
+            <child_frame_id>base_link</child_frame_id>
+            <odom_publisher_frequency>50</odom_publisher_frequency>
+            <tf_topic>/tf</tf_topic>
+        </plugin>
+        <plugin filename="gz-sim-joint-state-publisher-system"
+            name="gz::sim::systems::JointStatePublisher">
+            <topic>joint_states</topic>
+            <joint_name>left_rocker_joint</joint_name>
+            <joint_name>right_rocker_joint</joint_name>
+            <joint_name>left_bogie_joint</joint_name>
+            <joint_name>right_bogie_joint</joint_name>
+            <joint_name>diff_brace_joint</joint_name>
+            <joint_name>back_left_turnbuckle_joint</joint_name>
+            <joint_name>back_right_turnbuckle_joint</joint_name>
+            <joint_name>front_left_turnbuckle_joint</joint_name>
+            <joint_name>front_right_turnbuckle_joint</joint_name>
+            <joint_name>front_left_corner_joint</joint_name>
+            <joint_name>front_right_corner_joint</joint_name>
+            <joint_name>back_left_corner_joint</joint_name>
+            <joint_name>back_right_corner_joint</joint_name>
+        </plugin>
         <plugin filename="libgazebo_ros2_control.so" name="gazebo_ros2_control">
             <parameters>$(find rover_description)/config/control.yaml</parameters>

File: rover_description/urdf/bases/rocker.urdf.xacro (robot description, xacro)
@@ -23,5 +23,5 @@
     <xacro:property name="rocker_box_mass" value="0.25" />
     <xacro:include filename="$(find rover_description)/urdf/inertials.xacro"/>
-    <xacro:macro name="rocker" params="parent lat_label reflect">
+    <xacro:macro name="rocker" params="parent lat_label reflect use_gazebo:=true">
         <!-- link -->
         <link name="${lat_label}_rocker_link">
@@ -49,5 +49,7 @@
             <material>Gazebo/White</material>
         </gazebo>
-        <!-- joint -->
+        <!-- fix joint for simulation -->
+        <xacro:if value="${use_gazebo}">
+        <gazebo>
         <joint name="${lat_label}_rocker_joint" type="continuous">
             <origin rpy="0 0 0" xyz="0.071 ${reflect * 0.155} 0.0118"/>
@@ -61,4 +63,20 @@
             <child link="${lat_label}_rocker_link" />
         </joint>
+        </gazebo>
+        </xacro:if>
+        <!-- real joint for control -->
+        <xacro:unless value="${use_gazebo}">
+        <joint name="${lat_label}_rocker_joint" type="continuous">
+            <origin rpy="0 0 0" xyz="0.071 ${reflect * 0.155} 0.0118"/>
+            <axis xyz="0 1 0" />
+            <limit
+                lower="${-math_pi_over_4}"
+                upper="${math_pi_over_4}"
+                effort="100.0"
+                velocity="30.0" />
+            <parent link="${parent}" />
+            <child link="${lat_label}_rocker_link" />
+        </joint>
+        </xacro:unless>
         <gazebo reference="${lat_label}_rocker_joint">
             <provideFeedback>true</provideFeedback>

File: rover_description/urdf/bases/turnbuckle.urdf.xacro (robot description, xacro)
@@ -19,6 +19,5 @@
 <robot name="turnbuckle" xmlns:xacro="http://www.ros.org/wiki/xacro">
     <xacro:include filename="$(find rover_description)/urdf/inertials.xacro"/>
-    <xacro:macro name="turnbuckle" params="lat_label reflect">
-        <gazebo>
+    <xacro:macro name="turnbuckle" params="lat_label reflect use_gazebo:=true">
             <link name="${lat_label}_turnbuckle_link">
                 <pose>0.035 ${reflect * 0.17} 0.07 0 0 0</pose>
@@ -26,53 +25,42 @@
                     <pose>0 0 0 0 0 0</pose>
                     <geometry>
-                        <mesh>
-                            <uri>package://rover_description/meshes/bases/turnbuckle.stl</uri>
-                        </mesh>
-                        <!-- <cylinder>
-                            <length>0.07</length>
-                            <radius>0.0025</radius>
-                        </cylinder> -->
+                        <mesh filename="package://rover_description/meshes/bases/turnbuckle.stl"/>
                     </geometry>
-                    <material>
-                        <script>
-                            <uri>file://media/materials/scripts/gazebo.material</uri>
-                            <name>Gazebo/Blue</name>
-                        </script>
-                    </material>
                 </visual>
                 <collision name="${lat_label}_turnbuckle_collision">
                     <pose>0 0 0 0 ${math_pi_over_2} 0</pose>
                     <geometry>
-                        <cylinder>
-                            <length>0.07</length>
-                            <radius>0.0025</radius>
-                        </cylinder>
+                        <cylinder length="0.07" radius="0.0025"/>
                     </geometry>
                 </collision>
-                <inertial>
-                    <mass>0.01</mass>
-                    <inertia>
-                        <ixx>0.0001</ixx>
-                        <ixy>0</ixy>
-                        <ixz>0</ixz>
-                        <iyy>0.0001</iyy>
-                        <iyz>0</iyz>
-                        <izz>0.0001</izz>
-                    </inertia>
-                </inertial>
             </link>
-            <!-- can't have closed loops in URDF
-            <joint name="back_${lat_label}_turnbuckle_joint" type="ball">
-                <pose>-0.035 0 0 0 0 0</pose>
-                <parent>diff_brace_link</parent>
-                <child>${lat_label}_turnbuckle_link</child>
-            </joint>
-            -->
-            <joint name="front_${lat_label}_turnbuckle_joint" type="ball">
-                <pose>0.035 0 0 0 0 0</pose>
-                <parent>${lat_label}_rocker_link</parent>
-                <child>${lat_label}_turnbuckle_link</child>
-            </joint>
-        </gazebo>
+            <xacro:if value="${use_gazebo}">
+                <!-- can't have closed loops in URDF -->
+                <joint name="back_${lat_label}_turnbuckle_joint" type="fixed">
+                    <pose>-0.035 0 0 0 0 0</pose>
+                    <parent>diff_brace_link</parent>
+                    <child>${lat_label}_turnbuckle_link</child>
+                </joint>
+                <!--
+                <joint name="front_${lat_label}_turnbuckle_joint" type="fixed">
+                    <pose>0.035 0 0 0 0 0</pose>
+                    <parent>${lat_label}_rocker_link</parent>
+                    <child>${lat_label}_turnbuckle_link</child>
+                </joint>
+                -->
+            </xacro:if>
+            <xacro:unless value="${use_gazebo}">
+                <!-- can't have closed loops in URDF -->
+                <joint name="back_${lat_label}_turnbuckle_joint" type="ball">
+                    <pose>-0.035 0 0 0 0 0</pose>
+                    <parent>diff_brace_link</parent>
+                    <child>${lat_label}_turnbuckle_link</child>
+                </joint>
+                <joint name="front_${lat_label}_turnbuckle_joint" type="ball">
+                    <pose>0.035 0 0 0 0 0</pose>
+                    <parent>${lat_label}_rocker_link</parent>
+                    <child>${lat_label}_turnbuckle_link</child>
+                </joint>
+            </xacro:unless>
     </xacro:macro>
 </robot>
