Commit message: more gazebo changes

File: rover_description/models/rover.urdf.xacro (robot description, xacro)
@@ -28,5 +28,5 @@
     </link>
     <gazebo reference="base_link">
-        <material>Gazebo/Orange</material>
+        <material>orange</material>
     </gazebo>
     <!-- body -->
@@ -95,5 +95,5 @@
     </plugin>
   </gazebo>
-    <ros2_control name="RoverSystem" type="system">
+  <ros2_control name="RoverSystem" type="system">
         <hardware>
             <plugin>gz_ros2_control/GazeboSimSystem</plugin>
@@ -197,5 +197,20 @@
             <state_interface name="effort"/>
         </joint>
-    </ros2_control>
+        <!--
+        <joint name="right_rocker_joint">
+            <state_interface name="position"/>
+            <state_interface name="effort"/>
+        </joint>
+        <joint name="left_rocker_joint">
+            <state_interface name="position"/>
+            <state_interface name="effort"/>
+        </joint>
+        <joint name="diff_brace_joint">
+            <state_interface name="position"/>
+            <state_interface name="velocity"/>
+            <state_interface name="effort"/>
+        </joint>
+        -->
+  </ros2_control>
 <!-- Plugin config from https://github.com/ThiwakarS/ROS2-jazzy-GZ-harmonic -->
 <!--
@@ -212,5 +227,4 @@
             filename="gz-sim-sensors-system"
             name="gz::sim::systems::Sensors">
-            <render_engine>ogre2</render_engine>
         </plugin>
         <plugin

File: rover_description/urdf/bases/body.urdf.xacro (robot description, xacro)
@@ -46,5 +46,5 @@
         </link>
         <gazebo reference="body_box_link">
-            <material>Gazebo/White</material>
+            <material name="white" />
         </gazebo>
         <joint name="body_box_joint" type="fixed">

File: rover_description/urdf/bases/bogie.urdf.xacro (robot description, xacro)
@@ -46,5 +46,5 @@
         </link>
         <gazebo reference="${lat_label}_bogie_link">
-            <material>Gazebo/White</material>
+            <material name="white" />
         </gazebo>
         <!-- joint -->
@@ -55,8 +55,9 @@
                 lower="${-math_pi_over_4}"
                 upper="${math_pi_over_4}"
-                effort="100.0"
-                velocity="30.0" />
+                effort="0.0"
+                velocity="0.0" />
             <parent link="${lat_label}_rocker_link" />
             <child link="${lat_label}_bogie_link" />
+            <dynamics damping="0.05" friction="0.0"/>
         </joint>
         <gazebo reference="${lat_label}_bogie_joint">

File: rover_description/urdf/bases/differential.urdf.xacro (robot description, xacro)
@@ -27,8 +27,6 @@
             <visual>
                 <origin rpy="0 0 0" xyz="0 0 0" />
-                <!-- <origin rpy="0 0 ${math_pi_over_2}" xyz="0 0 0" /> -->
                 <geometry>
                     <mesh filename="package://rover_description/meshes/bases/differential.stl" />
-                    <!-- <box size="0.200 0.015 0.015"/> -->
                 </geometry>
                 <material name="white" />
@@ -46,5 +44,5 @@
         </link>
         <gazebo reference="diff_brace_link">
-            <material>Gazebo/White</material>
+            <material name="white" />
         </gazebo>
         <joint name="diff_brace_joint" type="revolute">
@@ -52,15 +50,13 @@
             <axis xyz="0 0 1" />
             <limit
-                lower="${-math_pi_over_4}"
-                upper="${math_pi_over_4}"
-                effort="100.0"
-                velocity="30.0" />
+                lower="-0.2"
+                upper="0.2"
+                effort="0.0"
+                velocity="0.0" />
             <parent link="${parent}" />
             <child link="diff_brace_link" />
+            <dynamics damping="1.0" friction="1.0"/>
+            <mimic joint="right_rocker_joint" multiplier="0.35" offset="0.0"/>
         </joint>
-        <gazebo reference="diff_brace_joint">
-            <provideFeedback>true</provideFeedback>
-            <implicitSpringDamper>true</implicitSpringDamper>
-        </gazebo>
     </xacro:macro>
 </robot>

File: rover_description/urdf/bases/rocker.urdf.xacro (robot description, xacro)
@@ -47,22 +47,27 @@
         </link>
         <gazebo reference="${lat_label}_rocker_link">
-            <material>Gazebo/White</material>
+            <material name="white" />
         </gazebo>
-        <joint name="${lat_label}_rocker_joint" type="continuous">
+        <!-- should be fixed for gazebo simulation, continuous for actual rover -->
+        <joint name="${lat_label}_rocker_joint" type="revolute"> <!-- fixed -->
             <origin rpy="0 0 0" xyz="0.071 ${reflect * 0.155} 0.0118"/>
             <axis xyz="0 1 0" />
             <limit
-                lower="${-math_pi_over_4}"
-                upper="${math_pi_over_4}"
-                effort="100.0"
-                velocity="30.0" />
+                lower="-0.3"
+                upper="0.3"
+                effort="0.0"
+                velocity="0.0" />
             <parent link="${parent}" />
             <child link="${lat_label}_rocker_link" />
-            <!-- In gazebo make the right rocker joint mimic the left.  In the Actual rover,
-                 this is done by the differential bars -->
+            <dynamics damping="0.05" friction="0.0"/>
+            <!-- Outside (i.e. RVIZ), you can make the rocker joints mimic the differential bar.
+                 In the Actual rover, this is done by the turnbuckles attached to the differential bar -->
+                 <!-- dist between center of rover and top end turnbuckle= 166.5 mm -->
+                 <!-- dist between pivot of rocker and other end of turnbuckle = 58 mm -->
             <xacro:if value="${use_gazebo}">
-                <xacro:if value="${lat_label == 'right'}">
-                    <mimic joint="left_rocker_joint" multiplier="-1.0" offset="0.0"/>
-                </xacro:if>
+              <xacro:if value="${lat_label == 'left'}">
+                <mimic joint="right_rocker_joint" multiplier="1" offset="0.0"/>
+              </xacro:if>
+                <!-- <mimic joint="diff_brace_joint" multiplier="-2.87" offset="0.0"/> -->
             </xacro:if>
         </joint>

File: rover_description/urdf/bases/turnbuckle.urdf.xacro (robot description, xacro)
@@ -20,27 +20,45 @@
     <xacro:include filename="$(find rover_description)/urdf/inertials.xacro"/>
     <xacro:macro name="turnbuckle" params="lat_label reflect use_gazebo:=true">
-        <gazebo>
             <link name="${lat_label}_turnbuckle_link">
-                <pose>0.035 ${reflect * 0.17} 0.07 0 0 0</pose>
                 <visual name="${lat_label}_turnbuckle_visual">
-                    <pose>0 0 0 0 0 0</pose>
+                    <origin xyz="0 0 0.035" rpy="${math_pi_over_2} ${math_pi_over_2} 0" />
                     <geometry>
                         <mesh filename="package://rover_description/meshes/bases/turnbuckle.stl"/>
                     </geometry>
+                    <material name="white" />
                 </visual>
                 <collision name="${lat_label}_turnbuckle_collision">
-                    <pose>0 0 0 0 ${math_pi_over_2} 0</pose>
+                    <origin xyz="0 0 0.035" rpy="0 0 0" />
                     <geometry>
-                        <cylinder length="0.07" radius="0.0025"/>
+                        <cylinder radius="0.0045" length="0.10" />
                     </geometry>
                 </collision>
+                   <xacro:solid_cylinder_inertial
+                    rpy="0 0 0" xyz="0 0 0"
+                    mass="0.25"
+                    radius="0.0025"
+                    length="0.07" />
             </link>
-            <xacro:if value="${use_gazebo}">
+            <!-- <xacro:unless value="${use_gazebo}"> -->
                 <!-- can't have closed loops in URDF -->
-                <joint name="back_${lat_label}_turnbuckle_joint" type="fixed">
-                    <pose>-0.035 0 0 0 0 0</pose>
-                    <parent>diff_brace_link</parent>
-                    <child>${lat_label}_turnbuckle_link</child>
+                <joint name="back_${lat_label}_turnbuckle_joint" type="revolute">
+                    <origin xyz="0 ${reflect * 0.17} 0" rpy="0 ${math_pi_over_2} 0" />
+                    <axis xyz="1 0 0" />
+                    <limit
+                        lower="${-math_pi}"
+                        upper="${math_pi}"
+                        effort="100.0"
+                        velocity="30.0" />
+                    <parent link="diff_brace_link" />
+                    <child link="${lat_label}_turnbuckle_link" />
+                    <xacro:if value="${lat_label == 'left'}">
+                      <mimic joint="right_rocker_joint" multiplier="0.35" offset="0.0"/>
+                    </xacro:if>
+                    <xacro:if value="${lat_label == 'right'}">
+                      <mimic joint="right_rocker_joint" multiplier="-0.35" offset="0.0"/>
+                    </xacro:if>
+                      <!-- <mimic joint="diff_brace_joint" multiplier="-2.87" offset="0.0"/> -->
                 </joint>
+    <gazebo>
                 <!--
                 <joint name="front_${lat_label}_turnbuckle_joint" type="fixed">
@@ -50,18 +68,5 @@
                 </joint>
                 -->
-            </xacro:if>
-            <xacro:unless value="${use_gazebo}">
-                <!-- can't have closed loops in URDF -->
-                <joint name="back_${lat_label}_turnbuckle_joint" type="ball">
-                    <pose>-0.035 0 0 0 0 0</pose>
-                    <parent>diff_brace_link</parent>
-                    <child>${lat_label}_turnbuckle_link</child>
-                </joint>
-                <joint name="front_${lat_label}_turnbuckle_joint" type="ball">
-                    <pose>0.035 0 0 0 0 0</pose>
-                    <parent>${lat_label}_rocker_link</parent>
-                    <child>${lat_label}_turnbuckle_link</child>
-                </joint>
-            </xacro:unless>
+            <!-- </xacro:unless> -->
     </gazebo>
     </xacro:macro>

File: rover_description/urdf/sensors/hokuyo.urdf.xacro (robot description, xacro)
@@ -44,5 +44,5 @@
     </link>
     <gazebo reference="${prefix}_base_link">
-      <material>Gazebo/DarkGrey</material>
+      <material name="dark_gray"/>
     </gazebo>
     <joint name="${prefix}_joint" type="fixed">
@@ -57,5 +57,4 @@
           filename="gz-sim-sensors-system"
           name="gz::sim::systems::Sensors">
-          <render_engine>ogre2</render_engine>
       </plugin>
     </gazebo>

File: rover_description/urdf/sensors/imu.urdf.xacro (robot description, xacro)
@@ -46,5 +46,5 @@
     </link>
     <gazebo reference="${prefix}_link">
-      <material>Gazebo/Blue</material>
+      <material name="blue"/>
     </gazebo>
     <!--

File: rover_description/urdf/wheels/corner.urdf.xacro (robot description, xacro)
@@ -47,5 +47,5 @@
         </link>
         <gazebo reference="${lon_label}_${lat_label}_corner_link">
-            <material>Gazebo/White</material>
+            <material name="white"/>
         </gazebo>
     </xacro:macro>

File: rover_description/urdf/wheels/wheel.urdf.xacro (robot description, xacro)
@@ -45,5 +45,5 @@
         </link>
         <gazebo reference="${lon_label}_${lat_label}_wheel_link">
-            <material>Gazebo/DarkGray</material>
+            <material name="dark_gray"/>
             <mu1>1.0</mu1>
             <mu2>1.0</mu2>
