Commit message: basic launch working

File: rover_description/models/rover.urdf.xacro (robot description, xacro)
@@ -69,6 +69,169 @@
     <xacro:corner_wheel_joint lon_label="back" lat_label="right" reflect="-1"/>
     <!-- For Gazebo Harmonic (Ignition/Gazebo >= Garden), use gz-sim-joint-state-publisher-system -->
-    <!--
     <gazebo>
+        <plugin filename="gz-sim-joint-state-publisher-system"
+            name="gz::sim::systems::JointStatePublisher">
+            <topic>joint_states</topic>
+            <joint_name>left_rocker_joint</joint_name>
+            <joint_name>right_rocker_joint</joint_name>
+            <joint_name>left_bogie_joint</joint_name>
+            <joint_name>right_bogie_joint</joint_name>
+            <joint_name>diff_brace_joint</joint_name>
+            <joint_name>back_left_turnbuckle_joint</joint_name>
+            <joint_name>back_right_turnbuckle_joint</joint_name>
+<!-- can't sim these joints - closed loop
+            <joint_name>front_left_turnbuckle_joint</joint_name>
+            <joint_name>front_right_turnbuckle_joint</joint_name>
+-->
+            <joint_name>front_left_corner_joint</joint_name>
+            <joint_name>front_right_corner_joint</joint_name>
+            <joint_name>back_left_corner_joint</joint_name>
+            <joint_name>back_right_corner_joint</joint_name>
+        </plugin>
+    </gazebo>
+  <ros2_control name="GazeboSystem" type="system">
+        <hardware>
+            <plugin>gz_ros2_control/GazeboSimSystem</plugin>
+        </hardware>
+        <joint name="front_right_corner_joint">
+            <command_interface name="position">
+                <param name="min">-3.14159</param>
+                <param name="max">3.14159</param>
+            </command_interface>
+            <state_interface name="position">
+                <param name="initial_value">0.0</param>
+            </state_interface>
+            <state_interface name="velocity"/>
+            <state_interface name="effort"/>
+        </joint>
+        <joint name="front_left_corner_joint">
+            <command_interface name="position">
+                <param name="min">-3.14159</param>
+                <param name="max">3.14159</param>
+            </command_interface>
+            <state_interface name="position">
+                <param name="initial_value">0.0</param>
+            </state_interface>
+            <state_interface name="velocity"/>
+            <state_interface name="effort"/>
+        </joint>
+        <joint name="back_right_corner_joint">
+            <command_interface name="position">
+                <param name="min">-3.14159</param>
+                <param name="max">3.14159</param>
+            </command_interface>
+            <state_interface name="position">
+                <param name="initial_value">0.0</param>
+            </state_interface>
+            <state_interface name="velocity"/>
+            <state_interface name="effort"/>
+        </joint>
+        <joint name="back_left_corner_joint">
+            <command_interface name="position">
+                <param name="min">-3.14159</param>
+                <param name="max">3.14159</param>
+            </command_interface>
+            <state_interface name="position">
+                <param name="initial_value">0.0</param>
+            </state_interface>
+            <state_interface name="velocity"/>
+            <state_interface name="effort"/>
+        </joint>
+        <joint name="front_right_wheel_joint">
+            <command_interface name="velocity">
+                <param name="min">-10</param>
+                <param name="max">10</param>
+            </command_interface>
+            <state_interface name="position"/>
+            <state_interface name="velocity"/>
+            <state_interface name="effort"/>
+        </joint>
+        <joint name="front_left_wheel_joint">
+            <command_interface name="velocity">
+                <param name="min">-10</param>
+                <param name="max">10</param>
+            </command_interface>
+            <state_interface name="position"/>
+            <state_interface name="velocity"/>
+            <state_interface name="effort"/>
+        </joint>
+        <joint name="mid_right_wheel_joint">
+            <command_interface name="velocity">
+                <param name="min">-10</param>
+                <param name="max">10</param>
+            </command_interface>
+            <state_interface name="position"/>
+            <state_interface name="velocity"/>
+            <state_interface name="effort"/>
+        </joint>
+        <joint name="mid_left_wheel_joint">
+            <command_interface name="velocity">
+                <param name="min">-10</param>
+                <param name="max">10</param>
+            </command_interface>
+            <state_interface name="position"/>
+            <state_interface name="velocity"/>
+            <state_interface name="effort"/>
+        </joint>
+        <joint name="back_right_wheel_joint">
+            <command_interface name="velocity">
+                <param name="min">-10</param>
+                <param name="max">10</param>
+            </command_interface>
+            <state_interface name="position"/>
+            <state_interface name="velocity"/>
+            <state_interface name="effort"/>
+        </joint>
+        <joint name="back_left_wheel_joint">
+            <command_interface name="velocity">
+                <param name="min">-10</param>
+                <param name="max">10</param>
+            </command_interface>
+            <state_interface name="position"/>
+            <state_interface name="velocity"/>
+            <state_interface name="effort"/>
+        </joint>
+  </ros2_control>
+  <gazebo>
+    <plugin filename="gz_ros2_control-system" name="gz_ros2_control::GazeboSimROS2ControlPlugin">
+      <parameters>$(find rover_description)/config/control.yaml</parameters>
+    </plugin>
+  </gazebo>
+<!-- Plugin config from https://github.com/ThiwakarS/ROS2-jazzy-GZ-harmonic -->
+<!--
+<gazebo>
+        <plugin
+            filename="gz-sim-user-commands-system"
+            name="gz::sim::systems::UserCommands">
+        </plugin>
+        <plugin
+            filename="gz-sim-scene-broadcaster-system"
+            name="gz::sim::systems::SceneBroadcaster">
+        </plugin>
+        <plugin
+            filename="gz-sim-sensors-system"
+            name="gz::sim::systems::Sensors">
+        </plugin>
+        <plugin
+            filename="gz-sim-imu-system"
+            name="gz::sim::systems::Imu">
+        </plugin>
+    </gazebo>
+-->
+    <!-- Temporary
+        <plugin
+            filename="gz-sim-diff-drive-system"
+            name="gz::sim::systems::DiffDrive">
+            <left_joint>mid_left_wheel_joint</left_joint>
+            <right_joint>mid_right_wheel_joint</right_joint>
+            <wheel_separation>0.0929</wheel_separation>
+            <wheel_radius>0.06</wheel_radius>
+            <topic>cmd_vel</topic>
+            <odom_topic>odom</odom_topic>
+            <frame_id>odom</frame_id>
+            <child_frame_id>base_link</child_frame_id>
+            <odom_publisher_frequency>50</odom_publisher_frequency>
+            <tf_topic>/tf</tf_topic>
+        </plugin>
         <plugin filename="gz-sim-joint-state-publisher-system"
             name="gz::sim::systems::JointStatePublisher">
@@ -88,182 +251,4 @@
             <joint_name>back_right_corner_joint</joint_name>
         </plugin>
-    </gazebo>
-    -->
-  <gazebo>
-    <plugin filename="gz_ros2_control-system" name="gz_ros2_control::GazeboSimROS2ControlPlugin">
-      <parameters>$(find rover_description)/config/control.yaml</parameters>
-    </plugin>
-  </gazebo>
-  <ros2_control name="RoverSystem" type="system">
-        <hardware>
-            <plugin>gz_ros2_control/GazeboSimSystem</plugin>
-        </hardware>
-        <joint name="front_right_corner_joint">
-            <command_interface name="position">
-                <param name="min">-3.14159</param>
-                <param name="max">3.14159</param>
-            </command_interface>
-            <state_interface name="position">
-                <param name="initial_value">0.0</param>
-            </state_interface>
-            <state_interface name="velocity"/>
-            <state_interface name="effort"/>
-        </joint>
-        <joint name="front_left_corner_joint">
-            <command_interface name="position">
-                <param name="min">-3.14159</param>
-                <param name="max">3.14159</param>
-            </command_interface>
-            <state_interface name="position">
-                <param name="initial_value">0.0</param>
-            </state_interface>
-            <state_interface name="velocity"/>
-            <state_interface name="effort"/>
-        </joint>
-        <joint name="back_right_corner_joint">
-            <command_interface name="position">
-                <param name="min">-3.14159</param>
-                <param name="max">3.14159</param>
-            </command_interface>
-            <state_interface name="position">
-                <param name="initial_value">0.0</param>
-            </state_interface>
-            <state_interface name="velocity"/>
-            <state_interface name="effort"/>
-        </joint>
-        <joint name="back_left_corner_joint">
-            <command_interface name="position">
-                <param name="min">-3.14159</param>
-                <param name="max">3.14159</param>
-            </command_interface>
-            <state_interface name="position">
-                <param name="initial_value">0.0</param>
-            </state_interface>
-            <state_interface name="velocity"/>
-            <state_interface name="effort"/>
-        </joint>
-        <joint name="front_right_wheel_joint">
-            <command_interface name="velocity">
-                <param name="min">-10</param>
-                <param name="max">10</param>
-            </command_interface>
-            <state_interface name="position"/>
-            <state_interface name="velocity"/>
-            <state_interface name="effort"/>
-        </joint>
-        <joint name="front_left_wheel_joint">
-            <command_interface name="velocity">
-                <param name="min">-10</param>
-                <param name="max">10</param>
-            </command_interface>
-            <state_interface name="position"/>
-            <state_interface name="velocity"/>
-            <state_interface name="effort"/>
-        </joint>
-        <joint name="mid_right_wheel_joint">
-            <command_interface name="velocity">
-                <param name="min">-10</param>
-                <param name="max">10</param>
-            </command_interface>
-            <state_interface name="position"/>
-            <state_interface name="velocity"/>
-            <state_interface name="effort"/>
-        </joint>
-        <joint name="mid_left_wheel_joint">
-            <command_interface name="velocity">
-                <param name="min">-10</param>
-                <param name="max">10</param>
-            </command_interface>
-            <state_interface name="position"/>
-            <state_interface name="velocity"/>
-            <state_interface name="effort"/>
-        </joint>
-        <joint name="back_right_wheel_joint">
-            <command_interface name="velocity">
-                <param name="min">-10</param>
-                <param name="max">10</param>
-            </command_interface>
-            <state_interface name="position"/>
-            <state_interface name="velocity"/>
-            <state_interface name="effort"/>
-        </joint>
-        <joint name="back_left_wheel_joint">
-            <command_interface name="velocity">
-                <param name="min">-10</param>
-                <param name="max">10</param>
-            </command_interface>
-            <state_interface name="position"/>
-            <state_interface name="velocity"/>
-            <state_interface name="effort"/>
-        </joint>
-        <!--
-        <joint name="right_rocker_joint">
-            <state_interface name="position"/>
-            <state_interface name="effort"/>
-        </joint>
-        <joint name="left_rocker_joint">
-            <state_interface name="position"/>
-            <state_interface name="effort"/>
-        </joint>
-        <joint name="diff_brace_joint">
-            <state_interface name="position"/>
-            <state_interface name="velocity"/>
-            <state_interface name="effort"/>
-        </joint>
-        -->
-  </ros2_control>
-<!-- Plugin config from https://github.com/ThiwakarS/ROS2-jazzy-GZ-harmonic -->
-<!--
-<gazebo>
-        <plugin
-            filename="gz-sim-user-commands-system"
-            name="gz::sim::systems::UserCommands">
-        </plugin>
-        <plugin
-            filename="gz-sim-scene-broadcaster-system"
-            name="gz::sim::systems::SceneBroadcaster">
-        </plugin>
-        <plugin
-            filename="gz-sim-sensors-system"
-            name="gz::sim::systems::Sensors">
-        </plugin>
-        <plugin
-            filename="gz-sim-imu-system"
-            name="gz::sim::systems::Imu">
-        </plugin>
-    </gazebo>
--->
-    <!-- Temporary
-        <plugin
-            filename="gz-sim-diff-drive-system"
-            name="gz::sim::systems::DiffDrive">
-            <left_joint>mid_left_wheel_joint</left_joint>
-            <right_joint>mid_right_wheel_joint</right_joint>
-            <wheel_separation>0.0929</wheel_separation>
-            <wheel_radius>0.06</wheel_radius>
-            <topic>cmd_vel</topic>
-            <odom_topic>odom</odom_topic>
-            <frame_id>odom</frame_id>
-            <child_frame_id>base_link</child_frame_id>
-            <odom_publisher_frequency>50</odom_publisher_frequency>
-            <tf_topic>/tf</tf_topic>
-        </plugin>
-        <plugin filename="gz-sim-joint-state-publisher-system"
-            name="gz::sim::systems::JointStatePublisher">
-            <topic>joint_states</topic>
-            <joint_name>left_rocker_joint</joint_name>
-            <joint_name>right_rocker_joint</joint_name>
-            <joint_name>left_bogie_joint</joint_name>
-            <joint_name>right_bogie_joint</joint_name>
-            <joint_name>diff_brace_joint</joint_name>
-            <joint_name>back_left_turnbuckle_joint</joint_name>
-            <joint_name>back_right_turnbuckle_joint</joint_name>
-            <joint_name>front_left_turnbuckle_joint</joint_name>
-            <joint_name>front_right_turnbuckle_joint</joint_name>
-            <joint_name>front_left_corner_joint</joint_name>
-            <joint_name>front_right_corner_joint</joint_name>
-            <joint_name>back_left_corner_joint</joint_name>
-            <joint_name>back_right_corner_joint</joint_name>
-        </plugin>
         <plugin filename="libgazebo_ros2_control.so" name="gazebo_ros2_control">
             <parameters>$(find rover_description)/config/control.yaml</parameters>

File: rover_description/urdf/bases/rocker.urdf.xacro (robot description, xacro)
@@ -67,5 +67,5 @@
             <xacro:if value="${use_gazebo}">
               <xacro:if value="${lat_label == 'left'}">
-                <mimic joint="right_rocker_joint" multiplier="1" offset="0.0"/>
+                <mimic joint="right_rocker_joint" multiplier="-1" offset="0.0"/>
               </xacro:if>
                 <!-- <mimic joint="diff_brace_joint" multiplier="-2.87" offset="0.0"/> -->

Commit message: removed mimic joints - now fixed for use_gazebo

File: rover_description/models/rover.urdf.xacro (robot description, xacro)
@@ -16,5 +16,6 @@
                robot_state_publisher on the real robot? -->
     <!-- do we even need this since we set it to default to true in rocker & turnbuckle? -->
-    <xacro:property name="use_gazebo" value="true"/>
+    <xacro:arg name="use_gazebo" default="true"/>
+    <xacro:property name="use_gazebo" value="$(arg use_gazebo)"/>
     <!-- The base link -->
     <link name="base_link">
@@ -33,10 +34,10 @@
     <xacro:body parent="base_link" />
     <xacro:differential parent="base_link" />
-    <xacro:turnbuckle lat_label="left" reflect="1"/>
-    <xacro:turnbuckle lat_label="right" reflect="-1"/>
-    <xacro:rocker parent="base_link" lat_label="left" reflect="1"/>
-    <xacro:rocker parent="base_link" lat_label="right" reflect="-1"/>
-    <xacro:bogie lat_label="left" reflect="1"/>
-    <xacro:bogie lat_label="right" reflect="-1"/>
+    <xacro:turnbuckle lat_label="left" reflect="1" use_gazebo="${use_gazebo}"/>
+    <xacro:turnbuckle lat_label="right" reflect="-1" use_gazebo="${use_gazebo}"/>
+    <xacro:rocker parent="base_link" lat_label="left" reflect="1" use_gazebo="${use_gazebo}"/>
+    <xacro:rocker parent="base_link" lat_label="right" reflect="-1" use_gazebo="${use_gazebo}"/>
+    <xacro:bogie lat_label="left" reflect="1" use_gazebo="${use_gazebo}" />
+    <xacro:bogie lat_label="right" reflect="-1" use_gazebo="${use_gazebo}" />
     <xacro:sensor_hokuyo prefix="laser" parent="base_link" min_angle="-1.0" max_angle="1.0">
         <origin xyz="0.17 0 0.005" rpy="0 0 0"/>
@@ -88,4 +89,10 @@
             <joint_name>back_left_corner_joint</joint_name>
             <joint_name>back_right_corner_joint</joint_name>
+            <joint_name>front_left_wheel_joint</joint_name>
+            <joint_name>front_right_wheel_joint</joint_name>
+            <joint_name>mid_left_wheel_joint</joint_name>
+            <joint_name>mid_right_wheel_joint</joint_name>
+            <joint_name>back_left_wheel_joint</joint_name>
+            <joint_name>back_right_wheel_joint</joint_name>
         </plugin>
     </gazebo>

File: rover_description/urdf/bases/bogie.urdf.xacro (robot description, xacro)
@@ -23,5 +23,5 @@
     <xacro:property name="bogie_box_mass" value="0.25" />
     <xacro:include filename="$(find rover_description)/urdf/inertials.xacro"/>
-    <xacro:macro name="bogie" params="lat_label reflect">
+    <xacro:macro name="bogie" params="lat_label reflect use_gazebo:=true">
         <!-- link -->
         <link name="${lat_label}_bogie_link">
@@ -48,6 +48,6 @@
             <material name="white" />
         </gazebo>
-        <!-- joint -->
-        <joint name="${lat_label}_bogie_joint" type="revolute">
+        <!-- joint - fixed in gazebo, revolute if outside -->
+        <joint name="${lat_label}_bogie_joint" type="${'fixed' if use_gazebo else 'revolute'}">
             <origin rpy="0 0 0" xyz="-0.181 ${reflect * 0.025} -0.062"/>
             <axis xyz="0 1 0" />

File: rover_description/urdf/bases/differential.urdf.xacro (robot description, xacro)
@@ -57,5 +57,8 @@
             <child link="diff_brace_link" />
             <dynamics damping="1.0" friction="1.0"/>
+            <!-- This makes sense for display_rover_description, but not simulation -->
+            <!--
             <mimic joint="right_rocker_joint" multiplier="0.35" offset="0.0"/>
+            -->
         </joint>
     </xacro:macro>

File: rover_description/urdf/bases/rocker.urdf.xacro (robot description, xacro)
@@ -50,25 +50,27 @@
         </gazebo>
         <!-- should be fixed for gazebo simulation, continuous for actual rover -->
-        <joint name="${lat_label}_rocker_joint" type="revolute"> <!-- fixed -->
+        <joint name="${lat_label}_rocker_joint" type="${'fixed' if use_gazebo else 'revolute'}">
             <origin rpy="0 0 0" xyz="0.071 ${reflect * 0.155} 0.0118"/>
             <axis xyz="0 1 0" />
             <limit
-                lower="-0.3"
-                upper="0.3"
-                effort="0.0"
-                velocity="0.0" />
+            lower="-0.3"
+            upper="0.3"
+            effort="0.0"
+            velocity="0.0" />
             <parent link="${parent}" />
             <child link="${lat_label}_rocker_link" />
             <dynamics damping="0.05" friction="0.0"/>
+            <!-- This makes sense for display_rover_description, but not simulation -->
             <!-- Outside (i.e. RVIZ), you can make the rocker joints mimic the differential bar.
                  In the Actual rover, this is done by the turnbuckles attached to the differential bar -->
                  <!-- dist between center of rover and top end turnbuckle= 166.5 mm -->
                  <!-- dist between pivot of rocker and other end of turnbuckle = 58 mm -->
+            <!--
             <xacro:if value="${use_gazebo}">
               <xacro:if value="${lat_label == 'left'}">
                 <mimic joint="right_rocker_joint" multiplier="-1" offset="0.0"/>
               </xacro:if>
-                <!-- <mimic joint="diff_brace_joint" multiplier="-2.87" offset="0.0"/> -->
             </xacro:if>
+            -->
         </joint>
         <gazebo reference="${lat_label}_rocker_joint">

File: rover_description/urdf/bases/turnbuckle.urdf.xacro (robot description, xacro)
@@ -52,4 +52,6 @@
                     <parent link="diff_brace_link" />
                     <child link="${lat_label}_turnbuckle_link" />
+                    <!-- This makes sense for display_rover_description, but not simulation -->
+                    <!--
                     <xacro:if value="${lat_label == 'left'}">
                       <mimic joint="right_rocker_joint" multiplier="0.35" offset="0.0"/>
@@ -58,5 +60,5 @@
                       <mimic joint="right_rocker_joint" multiplier="-0.35" offset="0.0"/>
                     </xacro:if>
-                      <!-- <mimic joint="diff_brace_joint" multiplier="-2.87" offset="0.0"/> -->
+                    -->
                 </joint>
     <gazebo>
