Commit message: adding camera, depth, and rgbd sensors

File: rover_description/urdf/sensors/asus_xtion.urdf.xacro (robot description, xacro)
@@ -61,95 +61,76 @@
       </inertial>
     </link>
+    <!-- REP 103-compliant optical frame: Z forward, X right, Y down.
+         In this model, camera_frame is already oriented as optical; we add
+         an explicit camera_optical_frame with identity transform for standard naming. -->
+    <joint name="camera_optical_frame_joint" type="fixed">
+      <origin xyz="0 0 0" rpy="0 0 0" />
+      <parent link="camera_frame" />
+      <child link="camera_optical_frame" />
+    </joint>
+    <link name="camera_optical_frame">
+      <inertial>
+        <mass value="0.0001" />
+        <origin xyz="0 0 0" />
+        <inertia ixx="1e-6" ixy="0.0" ixz="0.0"
+          iyy="1e-6" iyz="0.0"
+          izz="1e-6" />
+      </inertial>
+    </link>
+    <gazebo reference="${prefix}_link">
 <!--
-    <gazebo reference="${prefix}_link">
-      <sensor name="camera" type="depth">
+      <sensor name="camera" type="camera">
+        <always_on>true</always_on>
+        <update_rate>20</update_rate>
         <visualize>true</visualize>
-        <update_rate>30</update_rate>
+        <topic>camera/image</topic>
         <camera>
-          <horizontal_fov>${63.0*2*math_pi_over_2/180.0}</horizontal_fov>
+          <horizontal_fov>1.3962634</horizontal_fov>
           <image>
-            <format>B8G8R8</format>
             <width>640</width>
             <height>480</height>
+            <format>R8G8B8</format>
           </image>
           <clip>
-            <near>0.3</near>
-            <far>8.0</far>
+            <near>0.1</near>
+            <far>15</far>
           </clip>
-          <distortion>
-            <k1>0.00000001</k1>
-            <k2>0.00000001</k2>
-            <k3>0.00000001</k3>
-            <p1>0.00000001</p1>
-            <p2>0.00000001</p2>
-          </distortion>
+          <noise>
+            <type>gaussian</type>
+             Noise is sampled independently per pixel on each frame.
+                That pixel's noise value is added to each of its color
+                channels, which at that point lie in the range [0,1].
+            <mean>0.0</mean>
+            <stddev>0.007</stddev>
+          </noise>
+          <optical_frame_id>camera_frame</optical_frame_id>
+          <camera_info_topic>camera/camera_info</camera_info_topic>
         </camera>
-        <plugin name="depth_camera_controller" filename="libgazebo_ros_camera.so">
-          <ros>
-            <qos>
-              <topic name="/camera/camera_info">
-                <publisher>
-                  <reliability>best_effort</reliability>
-                </publisher>
-              </topic>
-              <topic name="/camera/image_raw">
-                <publisher>
-                  <reliability>best_effort</reliability>
-                </publisher>
-              </topic>
-              <topic name="/camera/image_raw/compressed">
-                <publisher>
-                  <reliability>best_effort</reliability>
-                </publisher>
-              </topic>
-              <topic name="/camera/image_raw/compressedDepth">
-                <publisher>
-                  <reliability>best_effort</reliability>
-                </publisher>
-              </topic>
-              <topic name="/camera/image_raw/theora">
-                <publisher>
-                  <reliability>best_effort</reliability>
-                </publisher>
-              </topic>
-              <topic name="/camera/points">
-                <publisher>
-                  <reliability>best_effort</reliability>
-                </publisher>
-              </topic>
-              <topic name="/camera/depth/camera_info">
-                <publisher>
-                  <reliability>best_effort</reliability>
-                </publisher>
-              </topic>
-              <topic name="/camera/depth/image_raw">
-                <publisher>
-                  <reliability>best_effort</reliability>
-                </publisher>
-              </topic>
-              <topic name="/camera/depth/image_raw/compressed">
-                <publisher>
-                  <reliability>best_effort</reliability>
-                </publisher>
-              </topic>
-              <topic name="/camera/depth/image_raw/compressedDepth">
-                <publisher>
-                  <reliability>best_effort</reliability>
-                </publisher>
-              </topic>
-              <topic name="/camera/depth/image_raw/theora">
-                <publisher>
-                  <reliability>best_effort</reliability>
-                </publisher>
-              </topic>
-            </qos>
-          </ros>
-          <frame_name>camera_frame</frame_name>
-          <min_depth>0.3</min_depth>
-          <max_depth>8.0</max_depth>
-        </plugin>
-      </sensor>
+    </sensor>
+-->
+    <sensor name="rgbd_camera" type="rgbd_camera">
+      <camera>
+        <horizontal_fov>1.25</horizontal_fov>
+        <image>
+          <!-- Match 2D camera resolution to keep CameraInfo consistent -->
+          <width>640</width>
+          <height>480</height>
+        </image>
+        <clip>
+          <near>0.3</near>
+          <far>15</far>
+        </clip>
+        <optical_frame_id>camera_optical_frame</optical_frame_id>
+      </camera>
+      <always_on>true</always_on>
+      <update_rate>20</update_rate>
+      <visualize>true</visualize>
+  <!-- Use base-only topic; Gazebo will create subtopics: image, depth_image, camera_info, points -->
+  <topic>camera/camera_rgbd</topic>
+  <gz_frame_id>camera_frame</gz_frame_id>
+      <!-- Publish RGBD CameraInfo on its own topic to avoid collision with 2D camera info -->
+      <camera_info_topic>camera/camera_rgbd/camera_info</camera_info_topic>
+    </sensor>
     </gazebo>
--->
   </xacro:macro>
 </robot>

File: rover_description/urdf/sensors/hokuyo.urdf.xacro (robot description, xacro)
@@ -58,4 +58,5 @@
           name="gz::sim::systems::Sensors">
       </plugin>
+      <render_engine>ogre2</render_engine>
     </gazebo>
     <gazebo reference="${prefix}_link">

Commit message: orient point cloud with rover

File: rover_description/urdf/sensors/asus_xtion.urdf.xacro (robot description, xacro)
@@ -61,13 +61,14 @@
       </inertial>
     </link>
-    <!-- REP 103-compliant optical frame: Z forward, X right, Y down.
-         In this model, camera_frame is already oriented as optical; we add
-         an explicit camera_optical_frame with identity transform for standard naming. -->
-    <joint name="camera_optical_frame_joint" type="fixed">
-      <origin xyz="0 0 0" rpy="0 0 0" />
+    <!-- Frame dedicated for point cloud publishing. Based on observation: the
+         cloud appears rotated relative to the
+         optical frame. Create a child frame with that rotation so the point
+         cloud's header frame matches its data axes. -->
+    <joint name="camera_pointcloud_frame_joint" type="fixed">
+      <origin xyz="0 0 0" rpy="${math_pi_over_2} -${math_pi_over_2} 0" />
       <parent link="camera_frame" />
-      <child link="camera_optical_frame" />
+      <child link="camera_pointcloud_frame" />
     </joint>
-    <link name="camera_optical_frame">
+    <link name="camera_pointcloud_frame">
       <inertial>
         <mass value="0.0001" />
@@ -79,34 +80,4 @@
     </link>
     <gazebo reference="${prefix}_link">
-<!--
-      <sensor name="camera" type="camera">
-        <always_on>true</always_on>
-        <update_rate>20</update_rate>
-        <visualize>true</visualize>
-        <topic>camera/image</topic>
-        <camera>
-          <horizontal_fov>1.3962634</horizontal_fov>
-          <image>
-            <width>640</width>
-            <height>480</height>
-            <format>R8G8B8</format>
-          </image>
-          <clip>
-            <near>0.1</near>
-            <far>15</far>
-          </clip>
-          <noise>
-            <type>gaussian</type>
-             Noise is sampled independently per pixel on each frame.
-                That pixel's noise value is added to each of its color
-                channels, which at that point lie in the range [0,1].
-            <mean>0.0</mean>
-            <stddev>0.007</stddev>
-          </noise>
-          <optical_frame_id>camera_frame</optical_frame_id>
-          <camera_info_topic>camera/camera_info</camera_info_topic>
-        </camera>
-    </sensor>
--->
     <sensor name="rgbd_camera" type="rgbd_camera">
       <camera>
@@ -121,13 +92,12 @@
           <far>15</far>
         </clip>
-        <optical_frame_id>camera_optical_frame</optical_frame_id>
+        <optical_frame_id>camera_pointcloud_frame</optical_frame_id>
       </camera>
       <always_on>true</always_on>
       <update_rate>20</update_rate>
       <visualize>true</visualize>
-  <!-- Use base-only topic; Gazebo will create subtopics: image, depth_image, camera_info, points -->
-  <topic>camera/camera_rgbd</topic>
-  <gz_frame_id>camera_frame</gz_frame_id>
-      <!-- Publish RGBD CameraInfo on its own topic to avoid collision with 2D camera info -->
+      <topic>camera/camera_rgbd</topic>
+      <!-- Publish point cloud in the dedicated frame to correct orientation -->
+      <gz_frame_id>camera_pointcloud_frame</gz_frame_id>
       <camera_info_topic>camera/camera_rgbd/camera_info</camera_info_topic>
     </sensor>

Commit message: correct pointcloud orientation

File: rover_description/urdf/sensors/asus_xtion.urdf.xacro (robot description, xacro)
@@ -20,10 +20,5 @@
   <xacro:macro name="sensor_asus_xtion" params="prefix parent *origin ">
     <xacro:property name="math_pi_over_2" value="1.5707963267948966" />
-    <joint name="${prefix}_joint" type="fixed">
-      <axis xyz="1 0 0"/>
-      <xacro:insert_block name="origin"/>
-      <parent link="${parent}"/>
-      <child link="${prefix}_link"/>
-    </joint>
+    <!-- Define camera_link with X fwd and Z up per REP-103 -->
     <link name="${prefix}_link">
       <visual>
@@ -47,10 +42,12 @@
       </inertial>
     </link>
-    <joint name="camera_frame_joint" type="fixed">
-      <origin xyz="0 0 0" rpy="-${math_pi_over_2} 0 -${math_pi_over_2}" />
-      <parent link="${prefix}_link" />
-      <child link="camera_frame" />
+    <joint name="${prefix}_joint" type="fixed">
+      <axis xyz="1 0 0"/>
+      <xacro:insert_block name="origin"/>
+      <parent link="${parent}"/>
+      <child link="${prefix}_link"/>
     </joint>
-    <link name="camera_frame">
+    <!-- Define camera_link_optical with z fwd and y down per REP-105 -->
+    <link name="${prefix}_link_optical">
       <inertial>
         <mass value="0.001" />
@@ -61,14 +58,14 @@
       </inertial>
     </link>
+    <joint name="${prefix}_frame_joint" type="fixed">
+      <origin xyz="0 0 0" rpy="-${math_pi_over_2} 0 -${math_pi_over_2}" />
+      <parent link="${prefix}_link" />
+      <child link="${prefix}_link_optical" />
+    </joint>
     <!-- Frame dedicated for point cloud publishing. Based on observation: the
-         cloud appears rotated relative to the
+         cloud appears rotated relative to th
          optical frame. Create a child frame with that rotation so the point
          cloud's header frame matches its data axes. -->
-    <joint name="camera_pointcloud_frame_joint" type="fixed">
-      <origin xyz="0 0 0" rpy="${math_pi_over_2} -${math_pi_over_2} 0" />
-      <parent link="camera_frame" />
-      <child link="camera_pointcloud_frame" />
-    </joint>
-    <link name="camera_pointcloud_frame">
+    <link name="${prefix}_pointcloud_frame">
       <inertial>
         <mass value="0.0001" />
@@ -79,10 +76,20 @@
       </inertial>
     </link>
+    <joint name="camera_pointcloud_frame_joint" type="fixed">
+      <!-- Rotate +90deg about Y so optical +Z -> pointcloud +X -->
+      <origin xyz="0 0 0" rpy="0 -${math_pi_over_2} ${math_pi_over_2}" />
+      <parent link="${prefix}_link_optical" />
+      <child link="camera_pointcloud_frame" />
+    </joint>
     <gazebo reference="${prefix}_link">
     <sensor name="rgbd_camera" type="rgbd_camera">
+      <always_on>true</always_on>
+      <update_rate>20</update_rate>
+      <visualize>true</visualize>
+      <topic>camera/camera_rgbd</topic>
+      <camera_info_topic>camera/camera_rgbd/camera_info</camera_info_topic>
       <camera>
         <horizontal_fov>1.25</horizontal_fov>
         <image>
-          <!-- Match 2D camera resolution to keep CameraInfo consistent -->
           <width>640</width>
           <height>480</height>
@@ -92,13 +99,6 @@
           <far>15</far>
         </clip>
-        <optical_frame_id>camera_pointcloud_frame</optical_frame_id>
+        <optical_frame_id>${prefix}_pointcloud_frame</optical_frame_id>
       </camera>
-      <always_on>true</always_on>
-      <update_rate>20</update_rate>
-      <visualize>true</visualize>
-      <topic>camera/camera_rgbd</topic>
-      <!-- Publish point cloud in the dedicated frame to correct orientation -->
-      <gz_frame_id>camera_pointcloud_frame</gz_frame_id>
-      <camera_info_topic>camera/camera_rgbd/camera_info</camera_info_topic>
     </sensor>
     </gazebo>

Commit message: VO working with mars world

File: rover_description/urdf/sensors/asus_xtion.urdf.xacro (robot description, xacro)
@@ -63,30 +63,21 @@
       <child link="${prefix}_link_optical" />
     </joint>
-    <!-- Frame dedicated for point cloud publishing. Based on observation: the
-         cloud appears rotated relative to th
-         optical frame. Create a child frame with that rotation so the point
-         cloud's header frame matches its data axes. -->
-    <link name="${prefix}_pointcloud_frame">
-      <inertial>
-        <mass value="0.0001" />
-        <origin xyz="0 0 0" />
-        <inertia ixx="1e-6" ixy="0.0" ixz="0.0"
-          iyy="1e-6" iyz="0.0"
-          izz="1e-6" />
-      </inertial>
-    </link>
-    <joint name="camera_pointcloud_frame_joint" type="fixed">
-      <!-- Rotate +90deg about Y so optical +Z -> pointcloud +X -->
-      <origin xyz="0 0 0" rpy="0 -${math_pi_over_2} ${math_pi_over_2}" />
-      <parent link="${prefix}_link_optical" />
-      <child link="camera_pointcloud_frame" />
-    </joint>
+    <!-- RGBD camera  -->
+        <!-- RGBD camera also publishes camera/depth/depth_image/points
+         The point cloud is mis-aligned - see
+         https://github.com/gazebosim/gz-sensors/issues/29#issuecomment-3113732696
+         Leaving this comment in case it becomes important later.
+         If you look in the commit history, I added a second camera just for
+         points that aligned the point cloud properly (according to rviz2), but
+         collapsed to a single camera when optimizing for performance.
+         It was camera_pointcloud_frame.
+         -->
     <gazebo reference="${prefix}_link">
-    <!-- RGB camera for RGB images and camera_info (optical frame)-->
-    <sensor name="rgb_camera" type="camera">
+    <sensor name="rgbd_camera" type="rgbd_camera">
       <always_on>true</always_on>
-      <update_rate>30</update_rate>
+      <update_rate>10</update_rate>
       <visualize>false</visualize>
-      <topic>camera/rgb/image_raw</topic>
+      <topic>camera/rgbd</topic>
+      <!-- append /camera_info /depth_image /image /points -->
       <camera>
         <horizontal_fov>1.25</horizontal_fov>
@@ -100,48 +91,12 @@
           <far>15</far>
         </clip>
-        <optical_frame_id>${prefix}_link_optical</optical_frame_id>
-      </camera>
-    </sensor>
-    <!-- Depth camera for depth images (optical frame)
-         Also publushes camera/depth/depth_image/points
-         But it's mis-aligned - see
-         https://github.com/gazebosim/gz-sensors/issues/29#issuecomment-3113732696
-         -->
-    <sensor name="depth_camera" type="depth_camera">
-      <always_on>true</always_on>
-      <update_rate>30</update_rate>
-      <visualize>false</visualize>
-      <topic>camera/depth/depth_image</topic>
-      <camera>
-        <horizontal_fov>1.25</horizontal_fov>
-        <image>
-          <width>640</width>
-          <height>480</height>
-        </image>
+        <depth_camera>
         <clip>
           <near>0.3</near>
           <far>15</far>
         </clip>
+        </depth_camera>
+        <!-- <optical_frame_id>${prefix}_rgbd_frame</optical_frame_id> -->
         <optical_frame_id>${prefix}_link_optical</optical_frame_id>
-      </camera>
-    </sensor>
-    <!-- RGBD camera for pointcloud only (pointcloud frame) -->
-    <sensor name="pointcloud_camera" type="rgbd_camera">
-      <always_on>true</always_on>
-      <update_rate>30</update_rate>
-      <visualize>false</visualize>
-      <topic>camera/pointcloud</topic>
-      <!-- append /camera_info /depth_image /image /points -->
-      <camera>
-        <horizontal_fov>1.25</horizontal_fov>
-        <image>
-          <width>640</width>
-          <height>480</height>
-        </image>
-        <clip>
-          <near>0.3</near>
-          <far>15</far>
-        </clip>
-        <optical_frame_id>${prefix}_pointcloud_frame</optical_frame_id>
       </camera>
     </sensor>
